Commit message: modify play envs and urdf

File: parkour_legged_gym/resources/robots/lite3/urdf/Lite3.urdf (robot description, URDF)
Before this commit: robot MiniLiteV3, 18 links, 17 joints
Links:
- link FL_HIP: geometry 
- link FL_SHANK: geometry collision box size=0.02 0.02 0.18
- link FL_THIGH: geometry collision box size=0.02 0.02 0.16
- link FR_HIP: geometry 
- link FR_SHANK: geometry collision box size=0.02 0.02 0.18
- link FR_THIGH: geometry collision box size=0.02 0.02 0.16
- link HL_HIP: geometry 
- link HL_SHANK: geometry collision box size=0.02 0.02 0.18
- link HL_THIGH: geometry collision box size=0.02 0.02 0.16
- link HR_HIP: geometry 
- link HR_SHANK: geometry collision box size=0.02 0.02 0.18
- link HR_THIGH: geometry collision box size=0.02 0.02 0.16
- link TORSO: geometry collision box size=0.35 0.184 0.08

Commit message: change urdf

File: parkour_legged_gym/resources/robots/lite3/urdf/Lite3.urdf (robot description, URDF)
Before this commit: robot MiniLiteV3, 18 links, 17 joints
Links:
- removed link INERTIA
- link FL_FOOT: mass 1E-12 -> 0.02; geometry collision sphere radius=0.022
- link FL_HIP: mass 0.428 -> 0.550; geometry collision mesh filename=../meshes/fl_hip.STL
- link FL_SHANK: mass 0.115 -> 0.153; geometry collision mesh filename=../meshes/fl_shank_collision.STL
- link FL_THIGH: mass 0.61 -> 0.86; geometry collision mesh filename=../meshes/fl_thigh.STL
- link FR_FOOT: mass 1E-12 -> 0.02; geometry collision sphere radius=0.022
- link FR_HIP: mass 0.428 -> 0.550; geometry collision mesh filename=../meshes/fr_hip.STL
- link FR_SHANK: mass 0.115 -> 0.153; geometry collision mesh filename=../meshes/fr_shank_collision.STL
- link FR_THIGH: mass 0.61 -> 0.86; geometry collision mesh filename=../meshes/fr_thigh.STL
- link HL_FOOT: mass 1E-12 -> 0.02; geometry collision sphere radius=0.022
- link HL_HIP: mass 0.428 -> 0.550; geometry collision mesh filename=../meshes/hl_hip.STL
- link HL_SHANK: mass 0.115 -> 0.153; geometry collision mesh filename=../meshes/hl_shank_collision.STL
- link HL_THIGH: mass 0.61 -> 0.86; geometry collision mesh filename=../meshes/hl_thigh.STL
- link HR_FOOT: mass 1E-12 -> 0.02; geometry collision sphere radius=0.022
- link HR_HIP: mass 0.428 -> 0.550; geometry collision mesh filename=../meshes/hr_hip.STL
- link HR_SHANK: mass 0.115 -> 0.153; geometry collision mesh filename=../meshes/hr_shank_collision.STL
- link HR_THIGH: mass 0.61 -> 0.86; geometry collision mesh filename=../meshes/hr_thigh.STL
- link TORSO: mass None -> 5.6056; geometry collision mesh filename=../meshes/torso.STL
Joints:
- removed joint FL_HipX
- removed joint FL_HipY
- removed joint FL_Knee
- removed joint FR_HipX
- removed joint FR_HipY
- removed joint FR_Knee
- removed joint HL_HipX
- removed joint HL_HipY
- removed joint HL_Knee
- removed joint HR_HipX
- removed joint HR_HipY
- removed joint HR_Knee
- removed joint Torso2Inertia
- added joint FL_HipX_joint: type revolute, parent TORSO, child FL_HIP, origin xyz=0.1745 0.062 0 rpy=0 0 0, axis -1 0 0, limit lower=-0.523 upper=0.523 effort=30 velocity=20
- added joint FL_HipY_joint: type revolute, parent FL_HIP, child FL_THIGH, origin xyz=0 0.09735 0 rpy=0 0 0, axis 0 -1 0, limit lower=-2.67 upper=0.314 effort=30 velocity=20
- added joint FL_Knee_joint: type revolute, parent FL_THIGH, child FL_SHANK, origin xyz=0 0 -0.20 rpy=0 0 0, axis 0 -1 0, limit lower=0.524 upper=2.792 effort=30 velocity=20
- added joint FR_HipX_joint: type revolute, parent TORSO, child FR_HIP, origin xyz=0.1745 -0.062 0 rpy=0 0 0, axis -1 0 0, limit lower=-0.523 upper=0.523 effort=30 velocity=20
- added joint FR_HipY_joint: type revolute, parent FR_HIP, child FR_THIGH, origin xyz=0 -0.09735 0 rpy=0 0 0, axis 0 -1 0, limit lower=-2.67 upper=0.314 effort=30 velocity=20
- added joint FR_Knee_joint: type revolute, parent FR_THIGH, child FR_SHANK, origin xyz=0 0 -0.20 rpy=0 0 0, axis 0 -1 0, limit lower=0.524 upper=2.792 effort=30 velocity=20
- added joint HL_HipX_joint: type revolute, parent TORSO, child HL_HIP, origin xyz=-0.1745 0.062 0 rpy=0 0 0, axis -1 0 0, limit lower=-0.523 upper=0.523 effort=30 velocity=20
- added joint HL_HipY_joint: type revolute, parent HL_HIP, child HL_THIGH, origin xyz=0 0.09735 0 rpy=0 0 0, axis 0 -1 0, limit lower=-2.67 upper=0.314 effort=30 velocity=20
- added joint HL_Knee_joint: type revolute, parent HL_THIGH, child HL_SHANK, origin xyz=0 0 -0.20 rpy=0 0 0, axis 0 -1 0, limit lower=0.524 upper=2.792 effort=30 velocity=20
- added joint HR_HipX_joint: type revolute, parent TORSO, child HR_HIP, origin xyz=-0.1745 -0.062 0 rpy=0 0 0, axis -1 0 0, limit lower=-0.523 upper=0.523 effort=30 velocity=20
- added joint HR_HipY_joint: type revolute, parent HR_HIP, child HR_THIGH, origin xyz=0 -0.09735 0 rpy=0 0 0, axis 0 -1 0, limit lower=-2.67 upper=0.314 effort=30 velocity=20
- added joint HR_Knee_joint: type revolute, parent HR_THIGH, child HR_SHANK, origin xyz=0 0 -0.20 rpy=0 0 0, axis 0 -1 0, limit lower=0.524 upper=2.792 effort=30 velocity=20
- joint FL_Ankle: origin xyz=0 0 -0.21 -> xyz=0 0 -0.21012
- joint FR_Ankle: origin xyz=0 0 -0.21 -> xyz=0 0 -0.21012
- joint HL_Ankle: origin xyz=0 0 -0.21 -> xyz=0 0 -0.21012
- joint HR_Ankle: origin xyz=0 0 -0.21 -> xyz=0 0 -0.21012

Commit message: setting for 6_13_lite3

File: parkour_legged_gym/resources/robots/lite3/urdf/Lite3.urdf (robot description, URDF)
Before this commit: robot Lite3, 17 links, 16 joints
Links:
- link FL_FOOT: geometry collision sphere radius=0.022; visual sphere radius=0.022
- link FL_HIP: geometry collision mesh filename=../meshes/fl_hip.STL; visual mesh filename=../meshes/fl_hip.STL
- link FL_SHANK: geometry collision mesh filename=../meshes/fl_shank_collision.STL; visual mesh filename=../meshes/fl_shank_collision.STL
- link FL_THIGH: geometry collision mesh filename=../meshes/fl_thigh.STL; visual mesh filename=../meshes/fl_thigh.STL
- link FR_FOOT: geometry collision sphere radius=0.022; visual sphere radius=0.022
- link FR_HIP: geometry collision mesh filename=../meshes/fr_hip.STL; visual mesh filename=../meshes/fr_hip.STL
- link FR_SHANK: geometry collision mesh filename=../meshes/fr_shank_collision.STL; visual mesh filename=../meshes/fr_shank_collision.STL
- link FR_THIGH: geometry collision mesh filename=../meshes/fr_thigh.STL; visual mesh filename=../meshes/fr_thigh.STL
- link HL_FOOT: geometry collision sphere radius=0.022; visual sphere radius=0.022
- link HL_HIP: geometry collision mesh filename=../meshes/hl_hip.STL; visual mesh filename=../meshes/hl_hip.STL
- link HL_SHANK: geometry collision mesh filename=../meshes/hl_shank_collision.STL; visual mesh filename=../meshes/hl_shank_collision.STL
- link HL_THIGH: geometry collision mesh filename=../meshes/hl_thigh.STL; visual mesh filename=../meshes/hl_thigh.STL
- link HR_FOOT: geometry collision sphere radius=0.022; visual sphere radius=0.022
- link HR_HIP: geometry collision mesh filename=../meshes/hr_hip.STL; visual mesh filename=../meshes/hr_hip.STL
- link HR_SHANK: geometry collision mesh filename=../meshes/hr_shank_collision.STL; visual mesh filename=../meshes/hr_shank_collision.STL
- link HR_THIGH: geometry collision mesh filename=../meshes/hr_thigh.STL; visual mesh filename=../meshes/hr_thigh.STL
- link TORSO: geometry collision mesh filename=../meshes/torso.STL; visual mesh filename=../meshes/torso.STL
